File: mini Inverter.kicad_pcb (KiCad board)
At the start: 2 copper layers, 152.5 x 75 mm, 89 parts, among them IC1 KP2122DP, IC3 ULN2003, J1 Conn_01x03_Pin, J2 Conn_01x05_Pin, K1 MountingHole_Pad, K2 MountingHole_Pad, K3 MountingHole_Pad, K4 MountingHole_Pad, K5 MountingHole_Pad, K6 MountingHole_Pad, U2 L7805, U3 ESP32-WROOM-32, U4 AMS1117

Commit message: 270826
Parts:
- moved R36 2.55 mm to (143.7, 121.3)
- moved R35 2.55 mm to (143.7, 123.9)
- moved R37 2.55 mm to (143.7, 118.7)
- moved U3 1.59 mm to (67.1, 100.6)
Routing:
- net +12V: track 167.1 -> 308.6 mm
- net +3V3: track 2.22 -> 66.3 mm, vias 0 -> 3
- net +5V: track 11.4 -> 63.3 mm
- net /IN6: track 0.00 -> 33.4 mm, vias 0 -> 2
- net /+12VR: track 18.9 -> 10.5 mm
- net /K6: track 38.9 -> 32.7 mm
- net GND: track 61.5 -> 63.5 mm
- net /K4: track 62.5 -> 60.5 mm
- net /DHT11: track 24.3 -> 26.1 mm
- net /IN5: track 32.4 -> 34.0 mm
- net /BUZZ: track 5.27 -> 3.65 mm
- net /TX: track 18.5 -> 16.9 mm
- net /RX: track 19.1 -> 17.4 mm
- net /IN1: track 33.9 -> 35.4 mm
- net /IN2: track 33.0 -> 34.6 mm
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- added copper zone on B.Cu, net GND
