File: mini Inverter.kicad_pcb (KiCad board)
At the start: 2 copper layers, 152.5 x 75 mm, 89 parts, among them IC1 KP2122DP, IC3 ULN2003, J1 Conn_01x03_Pin, J2 Conn_01x05_Pin, K1 MountingHole_Pad, K2 MountingHole_Pad, K3 MountingHole_Pad, K4 MountingHole_Pad, K5 MountingHole_Pad, K6 MountingHole_Pad, U2 L7805, U3 ESP32-WROOM-32, U4 AMS1117

Commit message: 3108
Routing:
- net /AC_LF1N: track 8.32 -> 2.30 mm
- net /AC_LF1L: track 8.71 -> 3.55 mm
