File: mini Inverter.kicad_sch (KiCad schematic)
At the start: 90 parts, among them IC1 KP2122DP, IC3 SOP16_IC, J1 Conn_01x03_Pin, J2 Conn_01x05_Pin, U1 LTV-817, U2 L7805, U3 ESP32-WROOM-32, U4 AMS1117

Commit message: 0408
Parts:
- IC3: value SOP16_IC -> ULN2003
Connections:
- net IN1: now also U3.33 (IO21); no longer U3.27 (IO16)
- net IN2: now also U3.31 (IO19); no longer U3.28 (IO17)
- net IN3: now also U3.30 (IO18); no longer U3.29 (IO5)
- net IN4: now also U3.29 (IO5); no longer U3.30 (IO18)
- net IN5: now also U3.28 (IO17); no longer U3.31 (IO19)
- net IN6: now also U3.27 (IO16); no longer U3.33 (IO21)
- net O1: now also IC3.15; no longer IC3.10
- net O2: now also IC3.14; no longer IC3.11
- net O3: now also IC3.13; no longer IC3.12
- net O4: now also IC3.12; no longer IC3.13
- net O5: now also IC3.11; no longer IC3.14
- net O6: now also IC3.10; no longer IC3.15
Changed lines of the file:
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@@
 		)
 	)
+	(label "O3"
+		(at 265.43 111.76 270)
+		(effects
+			(font
+				(size 1.27 1.27)
+			)
+			(justify right bottom)
+		)
+	)
 	(label "EN"
 		(at 227.33 38.1 0)
@@
 		)
 	)
+	(label "O4"
+		(at 262.89 111.76 270)
+		(effects
+			(font
+				(size 1.27 1.27)
+			)
+			(justify right bottom)
+		)
+	)
 	(label "RX"
 		(at 248.92 63.5 0)
@@
 	)
 	(label "O6"
-		(at 270.51 111.76 270)
+		(at 257.81 111.76 270)
 		(effects
 			(font
@@
 		)
 	)
+	(label "IN1"
+		(at 248.92 66.04 0)
+		(effects
+			(font
+				(size 1.27 1.27)
+			)
+			(justify left bottom)
+		)
+	)
 	(label "TX"
 		(at 248.92 60.96 0)
@@
 		)
 	)
-	(label "O4"
-		(at 265.43 111.76 270)
-		(effects
-			(font
-				(size 1.27 1.27)
-			)
-			(justify right bottom)
-		)
-	)
 	(label "IN3"
 		(at 262.89 101.6 90)
@@
 		)
 	)
-	(label "COM"
-		(at 171.45 148.59 0)
+	(label "IN4"
+		(at 248.92 76.2 0)
 		(effects
 			(font
@@
 		)
 	)
-	(label "IN2"
-		(at 248.92 78.74 0)
+	(label "IN6"
+		(at 248.92 81.28 0)
+		(effects
+			(font
+				(size 1.27 1.27)
+			)
+			(justify left bottom)
+		)
+	)
+	(label "COM"
+		(at 171.45 148.59 0)
 		(effects
 			(font
@@
 		)
 	)
-	(label "IN3"
-		(at 248.92 76.2 0)
+	(label "DHT11"
+		(at 248.92 83.82 0)
 		(effects
 			(font
@@
 		)
 	)
-	(label "DHT11"
-		(at 248.92 83.82 0)
+	(label "IN2"
+		(at 248.92 71.12 0)
 		(effects
 			(font
@@
 	)
 	(label "O1"
-		(at 257.81 111.76 270)
+		(at 270.51 111.76 270)
 		(effects
 			(font
@@
 		)
 	)
-	(label "IN1"
-		(at 248.92 81.28 0)
-		(effects
-			(font
-				(size 1.27 1.27)
-			)
-			(justify left bottom)
-		)
-	)
 	(label "AC_16A"
 		(at 179.07 163.83 0)
@@
 		)
 	)
-	(label "O5"
-		(at 267.97 111.76 270)
+	(label "IN3"
+		(at 248.92 73.66 0)
 		(effects
 			(font
 				(size 1.27 1.27)
 			)
-			(justify right bottom)
+			(justify left bottom)
 		)
 	)
@@
 		)
 	)
-	(label "IN6"
-		(at 248.92 66.04 0)
-		(effects
-			(font
-				(size 1.27 1.27)
-			)
-			(justify left bottom)
-		)
-	)
 	(label "TX"
 		(at 229.87 38.1 0)
@@
 		)
 	)
-	(label "IN5"
-		(at 248.92 71.12 0)
-		(effects
-			(font
-				(size 1.27 1.27)
-			)
-			(justify left bottom)
-		)
-	)
 	(label "IN1"
 		(at 257.81 101.6 90)
@@
 		)
 	)
-	(label "O3"
-		(at 262.89 111.76 270)
+	(label "O4"
+		(at 240.03 130.81 0)
 		(effects
 			(font
 				(size 1.27 1.27)
 			)
-			(justify right bottom)
+			(justify left bottom)
 		)
 	)
-	(label "O4"
-		(at 240.03 130.81 0)
+	(label "310v"
+		(at 40.64 16.51 0)
 		(effects
 			(font
@@
 		)
 	)
-	(label "IN4"
-		(at 248.92 73.66 0)
+	(label "IN5"
+		(at 248.92 78.74 0)
 		(effects
 			(font
@@
 		)
 	)
-	(label "310v"
-		(at 40.64 16.51 0)
+	(label "O2"
+		(at 267.97 111.76 270)
 		(effects
 			(font
 				(size 1.27 1.27)
 			)
-			(justify left bottom)
+			(justify right bottom)
 		)
 	)
-	(label "O2"
+	(label "O5"
 		(at 260.35 111.76 270)
 		(effects
@@
 			)
 		)
-		(property "Value" "SOP16_IC"
+		(property "Value" "ULN2003"
 			(at 260.096 116.078 0)
 			(hide yes)

Commit message: 1208
Parts:
- added K1, K2, K3, K4, K5, K6: MountingHole_Pad, 1_Mycustomfootprint:Touch_SF20, symbol Mechanical:MountingHole_Pad
Connections:
- net GND: now also U3.15 (GND)
- net at U3.12 (IO27): now also K4.1
- net at U3.13 (IO14): now also K3.1
- net at U3.14 (IO12): now also K2.1
- net at U3.16 (IO13): now also K1.1
- net at U3.8 (IO32): now also K6.1
- net at U3.9 (IO33): now also K5.1

Commit message: 1408
Parts:
- added C18: 104, Resistor_SMD:R_0805_2012Metric, symbol Device:C
Connections:
- net +3V3: now also C18.1
- net GND: now also C18.2
Changed lines of the file:
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@@
 	)
 	(junction
+		(at 203.2 49.53)
+		(diameter 0)
+		(color 0 0 0 0)
+	)
+	(junction
 		(at 147.32 59.69)
 		(diameter 0)
@@
 	)
 	(junction
+		(at 204.47 59.69)
+		(diameter 0)
+		(color 0 0 0 0)
+	)
+	(junction
 		(at 243.84 140.97)
 		(diameter 0)
@@
 	(wire
 		(pts
+			(xy 199.39 58.42) (xy 199.39 59.69)
+		)
+		(stroke
+			(width 0)
+			(type default)
+		)
+	)
+	(wire
+		(pts
 			(xy 133.35 176.53) (xy 133.35 180.34)
 		)
@@
 	(wire
 		(pts
+			(xy 199.39 59.69) (xy 204.47 59.69)
+		)
+		(stroke
+			(width 0)
+			(type default)
+		)
+	)
+	(wire
+		(pts
 			(xy 175.26 52.07) (xy 175.26 59.69)
 		)
@@
 	(wire
 		(pts
+			(xy 203.2 49.53) (xy 199.39 49.53)
+		)
+		(stroke
+			(width 0)
+			(type default)
+		)
+	)
+	(wire
+		(pts
 			(xy 118.11 59.69) (xy 109.22 59.69)
 		)
@@
 	(wire
 		(pts
+			(xy 199.39 49.53) (xy 199.39 50.8)
+		)
+		(stroke
+			(width 0)
+			(type default)
+		)
+	)
+	(wire
+		(pts
 			(xy 262.89 22.86) (xy 262.89 25.4)
 		)
@@
 					(unit 1)
 				)
+			)
+		)
+	)
+	(symbol
+		(lib_id "Device:C")
+		(at 199.39 54.61 0)
+		(unit 1)
+		(body_style 1)
+		(exclude_from_sim no)
+		(in_bom yes)
+		(on_board yes)
+		(in_pos_files yes)
+		(dnp no)
+		(property "Reference" "C18"
+			(at 195.326 52.324 0)
+			(show_name no)
+			(do_not_autoplace no)
+			(effects
+				(font
+					(size 1.27 1.27)
+				)
+				(justify left)
+			)
+		)
+		(property "Value" "104"
+			(at 195.58 56.896 0)
+			(show_name no)
+			(do_not_autoplace no)
+			(effects
+				(font
+					(size 1.27 1.27)
+				)
+				(justify left)
+			)
+		)
+		(property "Footprint" "Resistor_SMD:R_0805_2012Metric"
+			(at 200.3552 58.42 0)
+			(hide yes)
+			(show_name no)
+			(do_not_autoplace no)
+			(effects
+				(font
+					(size 1.27 1.27)
+				)
+			)
+		)
+		(property "Datasheet" ""
+			(at 199.39 54.61 0)
+			(hide yes)
+			(show_name no)
+			(do_not_autoplace no)
+			(effects
+				(font
+					(size 1.27 1.27)
+				)
+			)
+		)
+		(property "Description" "Unpolarized capacitor"
+			(at 199.39 54.61 0)
+			(hide yes)
+			(show_name no)
+			(do_not_autoplace no)
+			(effects
+				(font
+					(size 1.27 1.27)
+				)
+			)
+		)
+		(pin "2"
+		)
+		(pin "1"
+		)
+		(instances
+			(project "mini Inverter"
+				(path "/37d9edb3-3b82-4f0a-b5f8-8b86d1ed1264"
+					(reference "C18")
+					(unit 1)
+				)

Commit message: 1808
Parts:
- removed C20: 0805, Resistor_SMD:R_0805_2012Metric, symbol Device:C
- removed D4: 1N4007, Diode_SMD:D_SMA, symbol Diode:1N4007
- removed FR2: R, Resistor_THT:R_Axial_DIN0414_L11.9mm_D4.5mm_P15.24mm_Horizontal, symbol Device:R
- removed R19, R45: 0805, Resistor_SMD:R_0805_2012Metric, symbol Device:R
- removed R39: 1206, Resistor_SMD:R_1206_3216Metric, symbol Device:R
- removed U1: LTV-817, Package_DIP:DIP-4_W7.62mm, symbol Isolator:LTV-817
Connections:
- net ACN: now reaches AC_N1.1, AC_N2.1, AC_N3.1, AC_N4.1, AC_N5.1, AC_N6.1, C4.1, CX1.1, FR1.2, R1.1
- net K6: now reaches K6.1, U3.8 (IO32)
- net AC_RL2: now reaches AC_L2.1, RLY2.14
- net +12VR: now reaches R35.2, R36.2, R37.2, U2.1 (IN)
- net K5: now reaches K5.1, U3.9 (IO33)
- net AC_FUSE: now reaches C4.2, CX1.2, F2.1, LF1.2, R3.2
- net K2: now reaches K2.1, U3.14 (IO12)
- net AC_RL6: now reaches AC_L6.1, RLY6.14
- net K1: now reaches K1.1, U3.16 (IO13)
- net K3: now reaches K3.1, U3.13 (IO14)
- net AC_RL1: now reaches AC_L1.1, RLY1.14
- net AC_RL4: now reaches AC_L4.1, RLY4.14
- net AC_RL5: now reaches AC_L5.1, RLY5.14
- net AC_RL3: now reaches AC_L3.1, RLY3.14
- net K4: now reaches K4.1, U3.12 (IO27)
- net AC_L1: now reaches FR1.1, LF1.3
- net ACL: now reaches AC_L7.1, F1.1, F2.2
- net FB1 renamed AC_LF1N
- net FB2 renamed AC_LF1L
- no-connect marks 3 -> 2
Other:
- note removed: "ACL"
- note removed: "ACN"
- note removed: "MCU"
- moved on the sheet: C6, R35, R36, R37

Commit message: 2108
Parts:
- removed EC5: C_Polarized, Capacitor_THT:CP_Radial_D6.3mm_P2.50mm, symbol Device:C_Polarized
- RLY1, RLY2, RLY3, RLY4, RLY5, RLY6, T1: value (none) -> ~
Other:
- moved on the sheet: C15

Commit message: 280926
Parts:
- RLY1, RLY2, RLY3, RLY4, RLY5, RLY6, T1: value ~ -> (none)
