File: Mach_trai_tim/mach_trai_tim/khoiLED.kicad_sch (KiCad schematic)
At the start: 20 parts

Commit message: 021026
Parts:
- D1, D10, D2, D3, D4, D5, D6, D7, D8, D9: footprint LED_THT:LED_D5.0mm -> 1_Mycustomfootprint:LED_D5.0mm
Changed lines of the file:
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@@
 			)
 		)
-		(property "Footprint" "LED_THT:LED_D5.0mm"
+		(property "Footprint" "1_Mycustomfootprint:LED_D5.0mm"
 			(at 140.97 127 0)
 			(hide yes)
@@
 			)
 		)
-		(property "Footprint" "LED_THT:LED_D5.0mm"
+		(property "Footprint" "1_Mycustomfootprint:LED_D5.0mm"
 			(at 140.97 85.09 0)
 			(hide yes)
@@
 			)
 		)
-		(property "Footprint" "LED_THT:LED_D5.0mm"
+		(property "Footprint" "1_Mycustomfootprint:LED_D5.0mm"
 			(at 140.97 69.85 0)
 			(hide yes)
@@
 			)
 		)
-		(property "Footprint" "LED_THT:LED_D5.0mm"
+		(property "Footprint" "1_Mycustomfootprint:LED_D5.0mm"
 			(at 140.97 77.47 0)
 			(hide yes)
@@
 			)
 		)
-		(property "Footprint" "LED_THT:LED_D5.0mm"
+		(property "Footprint" "1_Mycustomfootprint:LED_D5.0mm"
 			(at 140.97 97.79 0)
 			(hide yes)
@@
 			)
 		)
-		(property "Footprint" "LED_THT:LED_D5.0mm"
+		(property "Footprint" "1_Mycustomfootprint:LED_D5.0mm"
 			(at 140.97 91.44 0)
 			(hide yes)
@@
 			)
 		)
-		(property "Footprint" "LED_THT:LED_D5.0mm"
+		(property "Footprint" "1_Mycustomfootprint:LED_D5.0mm"
 			(at 140.97 105.41 0)
 			(hide yes)
@@
 			)
 		)
-		(property "Footprint" "LED_THT:LED_D5.0mm"
+		(property "Footprint" "1_Mycustomfootprint:LED_D5.0mm"
 			(at 140.97 62.23 0)
 			(hide yes)
@@
 			)
 		)
-		(property "Footprint" "LED_THT:LED_D5.0mm"
+		(property "Footprint" "1_Mycustomfootprint:LED_D5.0mm"
 			(at 140.97 113.03 0)
 			(hide yes)
@@
 			)
 		)
-		(property "Footprint" "LED_THT:LED_D5.0mm"
+		(property "Footprint" "1_Mycustomfootprint:LED_D5.0mm"
 			(at 140.97 120.65 0)
 			(hide yes)
