File: Mach_trai_tim/mach_trai_tim/mach_trai_tim.kicad_pcb (KiCad board)
At the start: 2 copper layers, 32 parts, among them J1 Conn_01x02_Pin, U1 LM555, U2 4017

Commit message: 041026
Parts:
- J1: value Conn_01x02_Pin -> Screw_Terminal_01x02; footprint Connector_BarrelJack:BarrelJack_Horizontal -> 1_Mycustomfootprint:TerminalBlock_Phoenix_MKDS-1,5-2_1x02_P5.00mm_Horizontal
- RV1: value ~ -> 10K; footprint Potentiometer_THT:Potentiometer_Piher_PC-16_Single_Horizontal -> 1_Mycustomfootprint:Potentiometer_Bourns_3296W_Vertical
- U2: footprint Package_DIP:DIP-16_W7.62mm -> 1_Mycustomfootprint:DIP-16_W7.62mm
- moved R6 431.9 mm to (-263.0, 24.2)
- moved D4 431.4 mm to (-263.0, 29.2)
- moved R5 430.0 mm to (-235.8, -4.95)
- moved D2 429.9 mm to (-228.1, -29.1)
- moved D3 429.1 mm to (-235.8, 0.05)
- moved R4 428.8 mm to (-228.5, -24.1)
- moved C5 428.6 mm to (-284.8, 142.5), turned to 180 degrees
- moved R7 424.7 mm to (-284.6, 46.4)
- moved D5 423.8 mm to (-284.6, 51.4)
- moved J1 422.5 mm to (-285.0, 152.8), turned to 0 degrees
- moved D1 422.1 mm to (-253.8, -54.6)
- moved R3 420.8 mm to (-253.8, -49.6)
- moved D10 416.8 mm to (-284.6, -32.6), turned to 180 degrees
- moved R12 415.6 mm to (-284.7, -28.0), turned to 180 degrees
- moved R8 411.0 mm to (-306.3, 24.2)
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Connections:
- C1 pad 2: Net-(C1-Pad2) -> GND
- C2 pad 1: Net-(C1-Pad2) -> +9V
- C7 pad 2: Net-(C7-Pad2) -> GND
- C8 pad 1: Net-(C7-Pad2) -> +9V
- J1 pad 1: +9V -> GND
- J1 pad 2: GND -> +9V
Routing:
- net GND: track 0.00 -> 578.5 mm
- net +9V: track 0.00 -> 412.3 mm
- net /KHOILED/Q9: track 0.00 -> 218.5 mm
- net /KHOILED/Q8: track 0.00 -> 183.4 mm
- net Net-(U1-THRES): track 0.00 -> 138.9 mm
- net /KHOILED/Q7: track 0.00 -> 134.6 mm
- net Net-(R1-Pad1): track 0.00 -> 103.5 mm
- net /KHOILED/Q6: track 0.00 -> 103.4 mm
- net /KHOILED/Q1: track 0.00 -> 100.4 mm
- net Net-(U1-DISCH): track 0.00 -> 89.3 mm
- net /KHOILED/Q4: track 0.00 -> 73.4 mm
- net /KHOILED/Q5: track 0.00 -> 63.3 mm
- net /KHOILED/Q0: track 0.00 -> 55.8 mm
- net /KHOILED/Q2: track 0.00 -> 49.7 mm
- net /KHOILED/Q3: track 0.00 -> 44.1 mm
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Other:
- board outline added: 123.2 x 218.4 mm
- board text added: "5VDC"
