File: Mach_trai_tim/mach_trai_tim/mach_trai_tim.kicad_sch (KiCad schematic)
At the start: 12 parts, among them J1 Conn_01x02_Pin, U1 LM555, U2 4017

Commit message: 021026
Parts:
- removed C2, C4: 1uF, symbol Device:C_Small_US
- removed C3: 0.1uF, symbol Device:C_Small
- added C2: 0.1uF, 1_Mycustomfootprint:Cap_104_THT, symbol Device:C_Small
- added C7, C8: 1uF, 1_Mycustomfootprint:CP_Radial_D5.0mm_P2.50mm, symbol Device:C_Small_US
- C1: footprint (none) -> 1_Mycustomfootprint:Cap_104_THT
- C5, C6: footprint (none) -> 1_Mycustomfootprint:CP_Radial_D5.0mm_P2.50mm
- J1: footprint (none) -> Connector_BarrelJack:BarrelJack_Horizontal
Connections:
- net +9V: now also C7.1
- net GND: now also C2.2, C8.2
- net at C1.2: now also C2.1
- new net: C7.2, C8.1

Commit message: 041026
Parts:
- removed J1: Conn_01x02_Pin, Connector_BarrelJack:BarrelJack_Horizontal, symbol Connector:Conn_01x02_Pin
- added J1: Screw_Terminal_01x02, 1_Mycustomfootprint:TerminalBlock_Phoenix_MKDS-1,5-2_1x02_P5.00mm_Horizontal, symbol Connector:Screw_Terminal_01x02
- RV1: value (none) -> 10K; footprint Potentiometer_THT:Potentiometer_Piher_PC-16_Single_Horizontal -> 1_Mycustomfootprint:Potentiometer_Bourns_3296W_Vertical
- U2: footprint Package_DIP:DIP-16_W7.62mm -> 1_Mycustomfootprint:DIP-16_W7.62mm
Connections:
- net +9V: now also C2.1, C8.1, J1.2 (Pin_2)
- net GND: now also C1.2, C7.2, J1.1 (Pin_1)
Other:
- moved on the sheet: C1, C2, C7, C8
