File: Mach_trai_tim/mach_trai_tim.kicad_pcb (KiCad board)
At the start: 2 copper layers, 123.2 x 218.4 mm, 32 parts, among them J1 Screw_Terminal_01x02, U1 LM555, U2 4017

Commit message: 051026
Parts:
- moved C6 5.13 mm to (-303.4, -6.40)
- moved C7 2.81 mm to (-295.0, -17.2)
- moved R10 2.02 mm to (-338.7, -24.1)
- moved D1 2.00 mm to (-253.8, -52.6)
- moved R4 2.00 mm to (-230.5, -24.1)
- moved R3 1.98 mm to (-253.8, -47.6)
- moved R11 1.98 mm to (-315.4, -47.6), turned to 0 degrees
- moved D9 1.98 mm to (-315.4, -52.6), turned to 0 degrees
- moved C1 1.71 mm to (-295.0, -12.0)
- moved C8 1.57 mm to (-259.8, -13.0), turned to 90 degrees
- moved U1 0.44 mm to (-295.4, -4.00)
- moved D2 0.37 mm to (-228.5, -29.1)
- moved D8 0.25 mm to (-340.6, -29.1)
Routing:
- net GND: track 578.5 -> 784.6 mm
- net +9V: track 412.3 -> 518.1 mm, vias 0 -> 2
- net Net-(U1-DISCH): track 89.3 -> 126.6 mm, vias 0 -> 2
- net /KHOILED/Q1: track 100.4 -> 70.0 mm
- net /CLK: track 23.7 -> 16.9 mm
- net /KHOILED/Q8: track 183.4 -> 187.7 mm
- net /KHOILED/Q0: track 55.8 -> 53.8 mm
- net Net-(U1-THRES): track 138.9 -> 137.1 mm, vias 0 -> 2
- net /KHOILED/Q7: track 134.6 -> 136.3 mm
- net Net-(D10-K): track 5.56 -> 6.57 mm
- net Net-(D2-K): track 6.17 -> 7.00 mm
- net Net-(D8-K): track 5.96 -> 5.23 mm
- net /CLK1: track 31.9 -> 32.6 mm
- net Net-(R1-Pad1): track 103.5 -> 102.9 mm

Commit message: 1007051026
Parts:
- turned D10 to 0 degrees
Routing:
- net /KHOILED/Q9: track 218.9 -> 221.4 mm
- net Net-(D10-K): track 6.57 -> 7.30 mm
Changed lines of the file:
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@@
 	(footprint "1_Mycustomfootprint:LED_D5.0mm"
 		(layer "F.Cu")
-		(at -284.57 -32.58 180)
+		(at -284.57 -32.58)
 		(descr "LED, diameter 5.0mm, 2 pins, http://cdn-reichelt.de/documents/datenblatt/A500/LL-504BC2E-009.pdf, generated by kicad-footprint-generator")
 		(tags "LED")
@@
 		)
 		(property "Sim.Pins" "1=K 2=A"
-			(at 0 0 180)
+			(at 0 0 0)
 			(unlocked yes)
 			(layer "F.Fab")
@@
 		(duplicate_pad_numbers_are_jumpers no)
 		(fp_line
-			(start -2.56 -1.545)
-			(end -2.56 1.545)
+			(start -4.44968 0)
+			(end -3.44968 0)
 			(stroke
 				(width 0.3)
@@
 		)
 		(fp_line
-			(start -4.44968 0)
-			(end -3.44968 0)
+			(start -2.56 -1.545)
+			(end -2.56 1.545)
 			(stroke
 				(width 0.3)
@@
 		)
 		(fp_arc
-			(start 2.99 0)
-			(mid 0.801779 2.880495)
-			(end -2.56 1.54483)
+			(start -2.56 -1.54483)
+			(mid 0.801779 -2.880495)
+			(end 2.99 0)
 			(stroke
 				(width 0.3)
@@
 		)
 		(fp_arc
-			(start -2.56 -1.54483)
-			(mid 0.801779 -2.880495)
-			(end 2.99 0)
+			(start 2.99 0)
+			(mid 0.801779 2.880495)
+			(end -2.56 1.54483)
 			(stroke
 				(width 0.3)
@@
 		)
 		(fp_line
-			(start -2.5 -1.469694)
-			(end -2.5 1.469694)
+			(start -4.44968 0)
+			(end -3.44968 0)
 			(stroke
-				(width 0.1)
+				(width 0.05)
 				(type solid)
 			)
@@
 		)
 		(fp_line
-			(start -4.44968 0)
-			(end -3.44968 0)
+			(start -2.5 -1.469694)
+			(end -2.5 1.469694)
 			(stroke
-				(width 0.05)
+				(width 0.1)
 				(type solid)
 			)
@@
 		)
 		(pad "1" thru_hole roundrect
-			(at -1.27 0 180)
+			(at -1.27 0)
 			(size 1.3 1.3)
 			(drill 0.8)
@@
 		)
 		(pad "2" thru_hole circle
-			(at 1.27 0 180)
+			(at 1.27 0)
 			(size 1.3 1.3)
 			(drill 0.8)
@@
 	)
 	(segment
-		(start -281.58 -32.58)
-		(end -283.3 -32.58)
+		(start -285.84 -32.58)
+		(end -285.84 -31.84)
 		(width 0.3)
 		(layer "B.Cu")
@@
 	)
 	(segment
-		(start -280.865 -31.865)
-		(end -281.58 -32.58)
+		(start -285.84 -31.84)
+		(end -282.025 -28.025)
 		(width 0.3)
 		(layer "B.Cu")
@@
 	)
 	(segment
-		(start -280.865 -28.025)
-		(end -280.865 -31.865)
+		(start -282.025 -28.025)
+		(end -280.865 -28.025)
 		(width 0.3)
 		(layer "B.Cu")
@@
 	)
 	(segment
+		(start -283.3 -32.58)
+		(end -285.235 -34.515)
+		(width 0.2)
+		(layer "B.Cu")
+		(net "/KHOILED/Q9")
+	)
+	(segment
+		(start -287.775 -34.515)
+		(end -288.505 -35.245)
+		(width 0.2)
+		(layer "B.Cu")
+		(net "/KHOILED/Q9")
+	)
+	(segment
 		(start -305.2 27.2)
 		(end -303.6 28.8)
@@
 	(segment
 		(start -304.01 -50.75)
-		(end -285.84 -32.58)
+		(end -288.505 -35.245)
 		(width 0.2)
 		(layer "B.Cu")
@@
 		(width 0.2)
 		(layer "B.Cu")
+		(net "/KHOILED/Q9")
+	)
+	(segment
+		(start -285.235 -34.515)
+		(end -287.775 -34.515)
+		(width 0.2)
+		(layer "B.Cu")
