File: Mach_trai_tim - Copy/mach_trai_tim.kicad_pcb (KiCad board)
At the start: 2 copper layers, 123.2 x 218.4 mm, 32 parts, among them J1 Screw_Terminal_01x02, U1 LM555, U2 4017

Commit message: 061026
Parts:
- moved D6 504.0 mm to (-306.3, 29.2)
- moved D7 504.0 mm to (-333.5, 0.05)
- moved C6 503.6 mm to (-303.4, -6.40)
- moved D8 503.5 mm to (-340.6, -29.1)
- moved R12 503.2 mm to (-284.7, -28.0)
- moved D10 503.2 mm to (-284.6, -32.6)
- moved C8 503.1 mm to (-259.8, -13.0)
- moved D1 503.1 mm to (-253.8, -52.6)
- moved D5 503.1 mm to (-284.6, 51.4)
- moved J1 503.1 mm to (-285.0, 152.8)
- moved R1 503.1 mm to (-284.8, 1.60)
- moved R10 503.1 mm to (-338.7, -24.1)
- moved R2 503.1 mm to (-284.8, 7.80)
- moved R3 503.1 mm to (-253.8, -47.6)
- moved R5 503.1 mm to (-235.8, -4.95)
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Routing:
- net GND: track 737.0 -> 784.6 mm
- net +9V: track 494.0 -> 518.1 mm
- net /KHOILED/Q8: track 179.8 -> 187.7 mm
- net Net-(D10-K): track 12.0 -> 7.30 mm
- net /KHOILED/Q9: track 217.3 -> 221.4 mm
- net Net-(U1-THRES): track 135.2 -> 137.1 mm
- net /KHOILED/Q5: track 64.9 -> 63.1 mm
- net Net-(D6-K): track 7.59 -> 6.05 mm
- net Net-(U1-DISCH): track 125.3 -> 126.6 mm
- net /KHOILED/Q1: track 68.8 -> 70.0 mm
- net Net-(R1-Pad1): track 101.8 -> 102.9 mm
- net Net-(D2-K): track 8.06 -> 7.00 mm
- net /KHOILED/Q6: track 104.2 -> 103.2 mm
- removed copper zone on B.Cu, net GND
