File: PCB_5RELAY/mini Inverter.kicad_pcb (KiCad board)
At the start: 2 copper layers, 152.5 x 75 mm, 89 parts, among them IC1 KP2122DP, IC3 ULN2003, J1 Conn_01x03_Pin, J2 Conn_01x05_Pin, K1 MountingHole_Pad, K2 MountingHole_Pad, K3 MountingHole_Pad, K4 MountingHole_Pad, K5 MountingHole_Pad, K6 MountingHole_Pad, U2 L7805, U3 ESP32-WROOM-32, U4 AMS1117

Commit message: 08071026
Parts:
- removed K1, K2, K3, K4, K5, K6: MountingHole_Pad, 1_Mycustomfootprint:Touch_SF20
Connections:
- U3 pad 12: /K4 -> unconnected-(U3-IO27-Pad12)
- U3 pad 13: /K3 -> unconnected-(U3-IO14-Pad13)
- U3 pad 14: /K2 -> unconnected-(U3-IO12-Pad14)
- U3 pad 16: /K1 -> unconnected-(U3-IO13-Pad16)
- U3 pad 8: /K6 -> unconnected-(U3-IO32-Pad8)
- U3 pad 9: /K5 -> unconnected-(U3-IO33-Pad9)
Routing:
- net /K4: track 60.5 -> 0.00 mm, vias 1 -> 0
- net /K3: track 54.4 -> 0.00 mm, vias 1 -> 0
- net /K5: track 45.2 -> 0.00 mm, vias 1 -> 0
- net /K6: track 32.7 -> 0.00 mm, vias 1 -> 0
- net /K2: track 32.5 -> 0.00 mm, vias 1 -> 0
- net /K1: track 11.5 -> 0.00 mm
- net /DHT11: track 26.1 -> 23.2 mm
